Commit message: Update eof model config

File: ur_description/urdf/inc/eof_small.xacro (robot description, xacro)
@@ -9,5 +9,5 @@
       <child link="${prefix}eof"/>
       <!-- The tool is directly attached to the flange. -->
-    	<origin rpy="0 0 1.57" xyz="0 0 0.05"/>
+    	<origin rpy="0 0 -1.57" xyz="0 0 0.05"/>
     </joint>
     <link name="${prefix}eof">
