Commit message: Fixed ur3e srdf naming and added world frame to ur_macro

File: ur_description/urdf/inc/ur_macro.xacro (robot description, xacro)
@@ -289,4 +289,11 @@
       <dynamics damping="0" friction="0"/>
     </joint>
+    <!-- define the ur's position and orientation in the world coordinate system -->
+    <link name="${prefix}world" />
+    <joint name="${prefix}world_joint" type="fixed">
+      <parent link="${prefix}world" />
+      <child link="${prefix}base_link" /> <!-- TODO: check base_link name of robot -->
+      <origin xyz="0.0 0.0 0.0" rpy="0.0 0.0 0.0" />
+    </joint>
     <!-- ROS-Industrial 'base' frame: base_link to UR 'Base' Coordinates transform -->
     <link name="${prefix}base"/>

Commit message: Added new package to support ur3e+inspire hand

File: ur_description/urdf/inc/ur_macro.xacro (robot description, xacro)
@@ -289,11 +289,4 @@
       <dynamics damping="0" friction="0"/>
     </joint>
-    <!-- define the ur's position and orientation in the world coordinate system -->
-    <link name="${prefix}world" />
-    <joint name="${prefix}world_joint" type="fixed">
-      <parent link="${prefix}world" />
-      <child link="${prefix}base_link" /> <!-- TODO: check base_link name of robot -->
-      <origin xyz="0.0 0.0 0.0" rpy="0.0 0.0 0.0" />
-    </joint>
     <!-- ROS-Industrial 'base' frame: base_link to UR 'Base' Coordinates transform -->
     <link name="${prefix}base"/>

File: ur_description/urdf/ur3e_with_eof_linear.xacro (robot description, xacro)
@@ -11,3 +11,11 @@
   <!-- TODO: check end-effector link name of robot -->
   <xacro:eof prefix="" connected_to="tool0"/>
+  <!--Define the robot poses in the world-->
+  <!-- define the ur's position and orientation in the world coordinate system -->
+  <link name="world" />
+  <joint name="world_joint" type="fixed">
+    <parent link="world" />
+    <child link="base_link" /> <!-- TODO: check base_link name of robot -->
+    <origin xyz="0.0 0.0 0.0" rpy="0.0 0.0 0.0" />
+  </joint>
 </robot>

File: ur_description/urdf/ur3e_with_inspire.xacro (robot description, xacro)
@@ -1,14 +1,14 @@
 <?xml version="1.0"?>
-<robot xmlns:xacro="http://ros.org/wiki/xacro" name="ur3e_with_eof">
-  <!-- ur5e -->
+<robot xmlns:xacro="http://ros.org/wiki/xacro" name="ur3e_with_inspire">
+  <!-- ur3e -->
   <xacro:include filename="$(find ur_description)/urdf/inc/ur3e_macro.xacro" />
   <!-- arm -->
   <xacro:ur3e_robot prefix="" />
   <!-- end-effector -->
-  <xacro:include filename="$(find ur_description)/urdf/inc/eof_small.xacro" />
+  <xacro:include filename="$(find ur_description)/urdf/inspire_hand_left.urdf.xacro" />
   <!-- end-effector -->
   <!-- Here we include the end-effector by setting the parameters -->
   <!-- TODO: check end-effector link name of robot -->
-  <xacro:eof prefix="" connected_to="tool0"/>
+  <xacro:inspire_hand_left prefix="" connected_to="tool0"/>
   <!--Define the robot poses in the world-->
   <!-- define the ur's position and orientation in the world coordinate system -->

File: ur_description/urdf/ur5e_with_eof.xacro (robot description, xacro)
@@ -11,3 +11,11 @@
   <!-- TODO: check end-effector link name of robot -->
   <xacro:eof prefix="" connected_to="tool0"/>
+  <!--Define the robot poses in the world-->
+  <!-- define the ur's position and orientation in the world coordinate system -->
+  <link name="world" />
+  <joint name="world_joint" type="fixed">
+    <parent link="world" />
+    <child link="base_link" /> <!-- TODO: check base_link name of robot -->
+    <origin xyz="0.0 0.0 0.0" rpy="0.0 0.0 0.0" />
+  </joint>
 </robot>
