Commit message: Updated dual_arm setup

File: ur_description/urdf/dual_arm.xacro (robot description, xacro)
@@ -1,8 +1,8 @@
 <?xml version="1.0"?>
-<robot xmlns:xacro="http://ros.org/wiki/xacro" name="dual_arm">
+<robot xmlns:xacro="http://ros.org/wiki/xacro" name="ur3e_with_inspire_dual_arm">
   <!-- ur3e -->
   <xacro:include filename="$(find ur_description)/urdf/inc/ur3e_macro.xacro" />
   <!-- right arm -->
-  <xacro:ur3e_robot prefix="right_" />
+  <xacro:ur3e_robot prefix="passive_" />
   <!-- end-effector -->
   <xacro:include filename="$(find ur_description)/urdf/inc/eof_small.xacro" />
@@ -10,7 +10,9 @@
   <!-- Here we include the end-effector by setting the parameters -->
   <!-- TODO: check end-effector link name of robot -->
-  <xacro:eof prefix="right_" connected_to="right_tool0"/>
+  <xacro:eof prefix="passive_" connected_to="passive_tool0"/>
+  <!-- ur3e -->
+  <xacro:include filename="$(find ur_description)/urdf/inc/ur3e_macro.xacro" />
   <!-- arm -->
-  <xacro:ur3e_robot prefix="left_" />
+  <xacro:ur3e_robot prefix="" />
   <!-- end-effector -->
   <xacro:include filename="$(find ur_description)/urdf/inspire_hand_left.urdf.xacro" />
@@ -18,16 +20,17 @@
   <!-- Here we include the end-effector by setting the parameters -->
   <!-- TODO: check end-effector link name of robot -->
-  <xacro:inspire_hand_left prefix="left_" connected_to="left_tool0"/>
-  <link name="world"/>
+  <xacro:inspire_hand_left prefix="" connected_to="tool0"/>
   <!--Define the robot poses in the world-->
+  <!-- define the ur's position and orientation in the world coordinate system -->
+  <link name="world" />
+  <joint name="world_joint" type="fixed">
+    <parent link="world" />
+    <child link="base_link" /> <!-- TODO: check base_link name of robot -->
+    <origin xyz="0.0 0.0 0.0" rpy="0.0 0.0 0.0" />
+  </joint>
   <joint name="world_to_right" type="fixed">
     <parent link="world" />
-    <child link = "right_base_link" />
+    <child link = "passive_base_link" />
     <origin xyz="-0.5 0 0" rpy="0 0 0" />
-  </joint>
-  <joint name="world_to_left" type="fixed">
-    <parent link="world" />
-    <child link = "left_base_link" />
-    <origin xyz="0.5 0 0" rpy="0 0 0" />
-  </joint>
+  <link name="world"/>
 </robot>

Commit message: Fixed format error

File: ur_description/urdf/dual_arm.xacro (robot description, xacro)
@@ -11,6 +11,4 @@
   <!-- TODO: check end-effector link name of robot -->
   <xacro:eof prefix="passive_" connected_to="passive_tool0"/>
-  <!-- ur3e -->
-  <xacro:include filename="$(find ur_description)/urdf/inc/ur3e_macro.xacro" />
   <!-- arm -->
   <xacro:ur3e_robot prefix="" />
@@ -32,5 +30,5 @@
     <parent link="world" />
     <child link = "passive_base_link" />
-    <origin xyz="-0.5 0 0" rpy="0 0 0" />
-  <link name="world"/>
+    <origin xyz="0.5 0 0" rpy="0 0 0" />
+  </joint>
 </robot>
