Commit message: Added package for dual arm

File: ur_description/urdf/dual_arm_left_with_inspire.xacro (robot description, xacro)
@@ -30,5 +30,5 @@
     <parent link="world" />
     <child link = "passive_base_link" />
-    <origin xyz="0.5 0 0" rpy="0 0 0" />
+    <origin xyz="0.685 0 0" rpy="0 0 0" />
   </joint>
 </robot>

File: ur_description/urdf/inspire_hand_left.urdf.xacro (robot description, xacro)
@@ -3,11 +3,11 @@
   <xacro:macro name="inspire_hand_left" params="prefix connected_to">
     <!--  joint limit reference: https://en.inspire-robots.com/-->
-    <joint name="hand_base_joint" type="fixed">
+    <joint name="${prefix}hand_base_joint" type="fixed">
       <!-- The parent link must be read from the robot model it is attached to. -->
       <parent link="${connected_to}"/>
-      <child link="hand_base_link"/>
+      <child link="${prefix}hand_base_link"/>
       <origin xyz="0 0 0" rpy="-1.5707963 0 -1.5707963"/>
     </joint>
-    <link name="hand_base_link">
+    <link name="${prefix}hand_base_link">
       <inertial>
         <origin xyz="-0.0025264 -0.066047 -0.0019598" rpy="0 0 0"/>
@@ -70,5 +70,5 @@
       </collision>
     </link>
-    <link name="thumb_proximal_base">
+    <link name="${prefix}thumb_proximal_base">
       <inertial>
         <origin xyz="0.0048817 0.0009382 -0.00722" rpy="0 0 0"/>
@@ -89,12 +89,12 @@
       </collision>
     </link>
-    <joint name="thumb_proximal_yaw_joint" type="revolute">
+    <joint name="${prefix}thumb_proximal_yaw_joint" type="revolute">
       <origin xyz="-0.01696 -0.0691 0.02045" rpy="1.5708 -1.5708 0"/>
-      <parent link="hand_base_link"/>
-      <child link="thumb_proximal_base"/>
+      <parent link="${prefix}hand_base_link"/>
+      <child link="${prefix}thumb_proximal_base"/>
       <axis xyz="0 0 1"/>
       <limit lower="0" upper="1.308" effort="1" velocity="0.5"/>
     </joint>
-    <link name="thumb_proximal">
+    <link name="${prefix}thumb_proximal">
       <inertial>
         <origin xyz="0.021932 -0.012785 -0.0080386" rpy="0 0 0"/>
@@ -115,12 +115,12 @@
       </collision>
     </link>
-    <joint name="thumb_proximal_pitch_joint" type="revolute">
+    <joint name="${prefix}thumb_proximal_pitch_joint" type="revolute">
       <origin xyz="0.0099867 0.0098242 -0.0089" rpy="-1.5708 0 0.16939"/>
-      <parent link="thumb_proximal_base"/>
-      <child link="thumb_proximal"/>
+      <parent link="${prefix}thumb_proximal_base"/>
+      <child link="${prefix}thumb_proximal"/>
       <axis xyz="0 0 -1"/>
       <limit lower="0" upper="0.6" effort="1" velocity="0.5"/>
     </joint>
-    <link name="thumb_intermediate">
+    <link name="${prefix}thumb_intermediate">
       <inertial>
         <origin xyz="0.0095544 0.0016282 -0.0071997" rpy="0 0 0"/>
@@ -141,13 +141,13 @@
       </collision>
     </link>
-    <joint name="thumb_intermediate_joint" type="revolute">
+    <joint name="${prefix}thumb_intermediate_joint" type="revolute">
       <origin xyz="0.04407 -0.034553 -0.0008" rpy="0 0 0"/>
-      <parent link="thumb_proximal"/>
-      <child link="thumb_intermediate"/>
+      <parent link="${prefix}thumb_proximal"/>
+      <child link="${prefix}thumb_intermediate"/>
       <axis xyz="0 0 -1"/>
       <limit lower="0" upper="0.8" effort="1" velocity="0.5"/>
-      <mimic joint="thumb_proximal_pitch_joint" multiplier="1.334" offset="0"/>
-    </joint>
-    <link name="thumb_distal">
+      <mimic joint="${prefix}thumb_proximal_pitch_joint" multiplier="1.334" offset="0"/>
+    </joint>
+    <link name="${prefix}thumb_distal">
       <inertial>
         <origin xyz="0.0092888 -0.0049529 -0.0060033" rpy="0 0 0"/>
@@ -168,13 +168,13 @@
       </collision>
     </link>
-    <joint name="thumb_distal_joint" type="revolute">
+    <joint name="${prefix}thumb_distal_joint" type="revolute">
       <origin xyz="0.020248 -0.010156 -0.0012" rpy="0 0 0"/>
-      <parent link="thumb_intermediate"/>
-      <child link="thumb_distal"/>
+      <parent link="${prefix}thumb_intermediate"/>
+      <child link="${prefix}thumb_distal"/>
       <axis xyz="0 0 -1"/>
       <limit lower="0" upper="0.4" effort="1" velocity="0.5"/>
-      <mimic joint="thumb_proximal_pitch_joint" multiplier="0.667" offset="0"/>
-    </joint>
-    <link name="index_proximal">
+      <mimic joint="${prefix}thumb_proximal_pitch_joint" multiplier="0.667" offset="0"/>
+    </joint>
+    <link name="${prefix}index_proximal">
       <inertial>
         <origin xyz="0.0012259 -0.011942 -0.0060001" rpy="0 0 0"/>
@@ -195,12 +195,12 @@
       </collision>
     </link>
-    <joint name="index_proximal_joint" type="revolute">
+    <joint name="${prefix}index_proximal_joint" type="revolute">
       <origin xyz="0.00028533 -0.13653 0.032268" rpy="-0.034907 0 0"/>
-      <parent link="hand_base_link"/>
-      <child link="index_proximal"/>
+      <parent link="${prefix}hand_base_link"/>
+      <child link="${prefix}index_proximal"/>
       <axis xyz="0 0 -1"/>
       <limit lower="0" upper="1.47" effort="1" velocity="0.5"/>
     </joint>
-    <link name="index_intermediate">
+    <link name="${prefix}index_intermediate">
       <inertial>
         <origin xyz="0.0019697 -0.019589 -0.005" rpy="0 0 0"/>
@@ -221,13 +221,13 @@
       </collision>
     </link>
-    <joint name="index_intermediate_joint" type="revolute">
+    <joint name="${prefix}index_intermediate_joint" type="revolute">
       <origin xyz="-0.0026138 -0.032026 -0.001" rpy="0 0 0"/>
-      <parent link="index_proximal"/>
-      <child link="index_intermediate"/>
+      <parent link="${prefix}index_proximal"/>
+      <child link="${prefix}index_intermediate"/>
       <axis xyz="0 0 -1"/>
       <limit lower="-0.04545" upper="1.56" effort="1" velocity="0.5"/>
-      <mimic joint="index_proximal_joint" multiplier="1.06399" offset="-0.04545"/>
-    </joint>
-    <link name="middle_proximal">
+      <mimic joint="${prefix}index_proximal_joint" multiplier="1.06399" offset="-0.04545"/>
+    </joint>
+    <link name="${prefix}middle_proximal">
       <inertial>
         <origin xyz="0.001297 -0.011934 -0.0060001" rpy="0 0 0"/>
@@ -248,12 +248,12 @@
       </collision>
     </link>
-    <joint name="middle_proximal_joint" type="revolute">
+    <joint name="${prefix}middle_proximal_joint" type="revolute">
       <origin xyz="0.00028533 -0.1371 0.01295" rpy="0 0 0"/>
-      <parent link="hand_base_link"/>
-      <child link="middle_proximal"/>
+      <parent link="${prefix}hand_base_link"/>
+      <child link="${prefix}middle_proximal"/>
       <axis xyz="0 0 -1"/>
       <limit lower="0" upper="1.47" effort="1" velocity="0.5"/>
     </joint>
-    <link name="middle_intermediate">
+    <link name="${prefix}middle_intermediate">
       <inertial>
         <origin xyz="0.001921 -0.020796 -0.005" rpy="0 0 0"/>
@@ -274,13 +274,13 @@
       </collision>
     </link>
-    <joint name="middle_intermediate_joint" type="revolute">
+    <joint name="${prefix}middle_intermediate_joint" type="revolute">
       <origin xyz="-0.0024229 -0.032041 -0.001" rpy="0 0 0"/>
-      <parent link="middle_proximal"/>
-      <child link="middle_intermediate"/>
+      <parent link="${prefix}middle_proximal"/>
+      <child link="${prefix}middle_intermediate"/>
       <axis xyz="0 0 -1"/>
       <limit lower="-0.04545" upper="1.56" effort="1" velocity="0.5"/>
-      <mimic joint="middle_proximal_joint" multiplier="1.06399" offset="-0.04545"/>
-    </joint>
-    <link name="ring_proximal">
+      <mimic joint="${prefix}middle_proximal_joint" multiplier="1.06399" offset="-0.04545"/>
+    </joint>
+    <link name="${prefix}ring_proximal">
       <inertial>
         <origin xyz="0.001297 -0.011934 -0.0060002" rpy="0 0 0"/>
@@ -301,12 +301,12 @@
       </collision>
     </link>
-    <joint name="ring_proximal_joint" type="revolute">
+    <joint name="${prefix}ring_proximal_joint" type="revolute">
       <origin xyz="0.00028533 -0.13691 -0.0062872" rpy="0.05236 0 0"/>
-      <parent link="hand_base_link"/>
-      <child link="ring_proximal"/>
+      <parent link="${prefix}hand_base_link"/>
+      <child link="${prefix}ring_proximal"/>
       <axis xyz="0 0 -1"/>
       <limit lower="0" upper="1.47" effort="1" velocity="0.5"/>
     </joint>
-    <link name="ring_intermediate">
+    <link name="${prefix}ring_intermediate">
       <inertial>
         <origin xyz="0.0021753 -0.019567 -0.005" rpy="0 0 0"/>
@@ -327,13 +327,13 @@
       </collision>
     </link>
-    <joint name="ring_intermediate_joint" type="revolute">
+    <joint name="${prefix}ring_intermediate_joint" type="revolute">
       <origin xyz="-0.0024229 -0.032041 -0.001" rpy="0 0 0"/>
-      <parent link="ring_proximal"/>
-      <child link="ring_intermediate"/>
+      <parent link="${prefix}ring_proximal"/>
+      <child link="${prefix}ring_intermediate"/>
       <axis xyz="0 0 -1"/>
       <limit lower="-0.04545" upper="1.56" effort="1" velocity="0.5"/>
-      <mimic joint="ring_proximal_joint" multiplier="1.06399" offset="-0.04545"/>
-    </joint>
-    <link name="pinky_proximal">
+      <mimic joint="${prefix}ring_proximal_joint" multiplier="1.06399" offset="-0.04545"/>
+    </joint>
+    <link name="${prefix}pinky_proximal">
       <inertial>
         <origin xyz="0.001297 -0.011934 -0.0060001" rpy="0 0 0"/>
@@ -354,12 +354,12 @@
       </collision>
     </link>
-    <joint name="pinky_proximal_joint" type="revolute">
+    <joint name="${prefix}pinky_proximal_joint" type="revolute">
       <origin xyz="0.00028533 -0.13571 -0.025488" rpy="0.10472 0 0"/>
-      <parent link="hand_base_link"/>
-      <child link="pinky_proximal"/>
+      <parent link="${prefix}hand_base_link"/>
+      <child link="${prefix}pinky_proximal"/>
       <axis xyz="0 0 -1"/>
       <limit lower="0" upper="1.47" effort="1" velocity="0.5"/>
     </joint>
-    <link name="pinky_intermediate">
+    <link name="${prefix}pinky_intermediate">
       <inertial>
         <origin xyz="0.0024748 -0.016203 -0.0050031" rpy="0 0 0"/>
@@ -380,41 +380,41 @@
       </collision>
     </link>
-    <joint name="pinky_intermediate_joint" type="revolute">
+    <joint name="${prefix}pinky_intermediate_joint" type="revolute">
       <origin xyz="-0.0024229 -0.032041 -0.001" rpy="0 0 0"/>
-      <parent link="pinky_proximal"/>
-      <child link="pinky_intermediate"/>
+      <parent link="${prefix}pinky_proximal"/>
+      <child link="${prefix}pinky_intermediate"/>
       <axis xyz="0 0 -1"/>
       <limit lower="-0.04545" upper="1.56" effort="1" velocity="0.5"/>
-      <mimic joint="pinky_proximal_joint" multiplier="1.06399" offset="-0.04545"/>
-    </joint>
-    <link name='thumb_tip'/>
-    <joint name="thumb_tip_joint" type="fixed">
+      <mimic joint="${prefix}pinky_proximal_joint" multiplier="1.06399" offset="-0.04545"/>
+    </joint>
+    <link name='${prefix}thumb_tip'/>
+    <joint name="${prefix}thumb_tip_joint" type="fixed">
       <origin xyz="0.0202 -0.0140 -0.006" rpy="0 0 0"/>
-      <parent link="thumb_distal"/>
-      <child link="thumb_tip"/>
-    </joint>
-    <link name='index_tip'/>
-    <joint name="index_tip_joint" type="fixed">
+      <parent link="${prefix}thumb_distal"/>
+      <child link="${prefix}thumb_tip"/>
+    </joint>
+    <link name='${prefix}index_tip'/>
+    <joint name="${prefix}index_tip_joint" type="fixed">
       <origin xyz="-0.0008 -0.045 -0.005" rpy="0 0 0"/>
-      <parent link="index_intermediate"/>
-      <child link="index_tip"/>
-    </joint>
-    <link name='middle_tip'/>
-    <joint name="middle_tip_joint" type="fixed">
+      <parent link="${prefix}index_intermediate"/>
+      <child link="${prefix}index_tip"/>
+    </joint>
+    <link name='${prefix}middle_tip'/>
+    <joint name="${prefix}middle_tip_joint" type="fixed">
       <origin xyz="-0.001 -0.048 -0.005" rpy="0 0 0"/>
-      <parent link="middle_intermediate"/>
-      <child link="middle_tip"/>
-    </joint>
-    <link name='ring_tip'/>
-    <joint name="ring_tip_joint" type="fixed">
+      <parent link="${prefix}middle_intermediate"/>
+      <child link="${prefix}middle_tip"/>
+    </joint>
+    <link name='${prefix}ring_tip'/>
+    <joint name="${prefix}ring_tip_joint" type="fixed">
       <origin xyz="-0.0008 -0.045 -0.005" rpy="0 0 0"/>
-      <parent link="ring_intermediate"/>
-      <child link="ring_tip"/>
-    </joint>
-    <link name='pinky_tip'/>
-    <joint name="pinky_tip_joint" type="fixed">
+      <parent link="${prefix}ring_intermediate"/>
+      <child link="${prefix}ring_tip"/>
+    </joint>
+    <link name='${prefix}pinky_tip'/>
+    <joint name="${prefix}pinky_tip_joint" type="fixed">
       <origin xyz="-0.0008 -0.037 -0.005" rpy="0 0 0"/>
-      <parent link="pinky_intermediate"/>
-      <child link="pinky_tip"/>
+      <parent link="${prefix}pinky_intermediate"/>
+      <child link="${prefix}pinky_tip"/>
     </joint>
   </xacro:macro>
