Commit message: Fixed urdf naming issue

File: ur_description/urdf/inspire_hand_v2_left.xacro (robot description, xacro)
@@ -650,5 +650,5 @@
   </joint>
   <link
-    name="${prefix}pinky_proximal_joint">
+    name="${prefix}left_little_1">
     <inertial>
       <origin
@@ -671,24 +671,24 @@
       <geometry>
         <mesh
-          filename="package://ur_description/meshes/inspire_hand/v2/pinky_proximal_joint.STL" />
-      </geometry>
-      <material
-        name="">
-        <color
-          rgba="0.792156862745098 0.819607843137255 0.933333333333333 1" />
-      </material>
-    </visual>
-    <collision>
-      <origin
-        xyz="0 0 0"
-        rpy="0 0 0" />
-      <geometry>
-        <mesh
-          filename="package://ur_description/meshes/inspire_hand/v2/pinky_proximal_joint.STL" />
-      </geometry>
-    </collision>
-  </link>
-  <joint
-    name="${prefix}pinky_proximal_joint_joint"
+          filename="package://ur_description/meshes/inspire_hand/v2/left_little_1.STL" />
+      </geometry>
+      <material
+        name="">
+        <color
+          rgba="0.792156862745098 0.819607843137255 0.933333333333333 1" />
+      </material>
+    </visual>
+    <collision>
+      <origin
+        xyz="0 0 0"
+        rpy="0 0 0" />
+      <geometry>
+        <mesh
+          filename="package://ur_description/meshes/inspire_hand/v2/left_little_1.STL" />
+      </geometry>
+    </collision>
+  </link>
+  <joint
+    name="${prefix}pinky_proximal_joint"
     type="revolute">
     <origin
@@ -698,5 +698,5 @@
       link="${prefix}hand_base_link" />
     <child
-      link="${prefix}pinky_proximal_joint" />
+      link="${prefix}left_little_1" />
     <axis
       xyz="0 0 -1" />
@@ -754,5 +754,5 @@
       rpy="0 0 0" />
     <parent
-      link="${prefix}pinky_proximal_joint" />
+      link="${prefix}left_little_1" />
     <child
       link="${prefix}left_little_2" />
@@ -765,5 +765,5 @@
       velocity="100" />
     <mimic
-        joint="${prefix}pinky_proximal_joint_joint"
+        joint="${prefix}pinky_proximal_joint"
         multiplier="1.05"
         offset="0" />
@@ -798,5 +798,5 @@
   <xacro:transmission_block joint_name="middle_proximal_joint"/>
   <xacro:transmission_block joint_name="ring_proximal_joint"/>
-  <xacro:transmission_block joint_name="pinky_proximal_joint_joint"/>
+  <xacro:transmission_block joint_name="pinky_proximal_joint"/>
   <xacro:macro name="mimic_joint_plugin_gazebo" params="name_prefix parent_joint mimic_joint has_pid:=false multiplier:=1.0 offset:=0 sensitiveness:=0.0 max_effort:=1.0 robot_namespace:=''">
     <gazebo>
@@ -833,5 +833,5 @@
     has_pid="true" multiplier="1.0" max_effort="10.0" />
   <xacro:mimic_joint_plugin_gazebo name_prefix="${prefix}left_little_2_joint"
-    parent_joint="${prefix}pinky_proximal_joint_joint" mimic_joint="${prefix}left_little_2_joint"
+    parent_joint="${prefix}pinky_proximal_joint" mimic_joint="${prefix}left_little_2_joint"
     has_pid="true" multiplier="1.0" max_effort="10.0" />
   </xacro:macro>
