Commit message: Added new setup for inspire hand_v2 right

File: ur_description/urdf/inspire_hand_v2_right.xacro (robot description, xacro)
@@ -1,9 +1,9 @@
 <?xml version="1.0" encoding="utf-8"?>
 <robot xmlns:xacro="http://www.ros.org/wiki/xacro">
-  <xacro:macro name="inspire_hand_left" params="prefix connected_to">
-    <joint name="${prefix}L_hand_base_joint" type="fixed">
-      <origin
-      xyz="-0.008 0.1132 0.112"
-      rpy="0 0 3.1415926" />
+  <xacro:macro name="inspire_hand_right" params="prefix connected_to">
+    <joint name="${prefix}R_hand_base_joint" type="fixed">
+      <origin
+      xyz="0.008 0.1132 0.112"
+      rpy="0 0 0" />
       <parent link="${connected_to}"/>
       <child link="${prefix}hand_base_link"/>
@@ -13,77 +13,77 @@
     <inertial>
       <origin
-        xyz="-0.00826856171690858 0.115495645683634 -0.0283405186091888"
-        rpy="0 0 0" />
-      <mass
-        value="0.260034351027079" />
-      <inertia
-        ixx="0.000223659755568991"
-        ixy="1.13436481431654E-06"
-        ixz="5.34309330483412E-07"
-        iyy="0.000266799681382808"
-        iyz="-1.40944118439409E-05"
-        izz="0.00013285776917007" />
-    </inertial>
-    <visual>
-      <origin
-        xyz="0 0 0"
-        rpy="0 0 0" />
-      <geometry>
-        <mesh
-          filename="package://ur_description/meshes/inspire_hand/v2/left/base_link.STL" />
-      </geometry>
-      <material
-        name="">
-        <color
-          rgba="0.792156862745098 0.819607843137255 0.933333333333333 1" />
-      </material>
-    </visual>
-    <collision>
-      <origin
-        xyz="0 0 0"
-        rpy="0 0 0" />
-      <geometry>
-        <mesh
-          filename="package://ur_description/meshes/inspire_hand/v2/left/base_link.STL" />
-      </geometry>
-    </collision>
-  </link>
-  <link
-    name="${prefix}left_thumb_swing">
-    <inertial>
-      <origin
-        xyz="-0.001897403655087 -7.12516796909923E-05 0.00313589310434412"
+        xyz="-0.00827757758571113 -0.0384721010257447 0.114789391580906"
+        rpy="0 0 0" />
+      <mass
+        value="0.314090908651444" />
+      <inertia
+        ixx="0.000240584294377349"
+        ixy="5.34716372850393E-07"
+        ixz="1.12900344118066E-06"
+        iyy="0.000155854672232219"
+        iyz="-1.41174523865224E-05"
+        izz="0.000284423438512345" />
+    </inertial>
+    <visual>
+      <origin
+        xyz="0 0 0"
+        rpy="0 0 0" />
+      <geometry>
+        <mesh
+          filename="package://ur_description/meshes/inspire_hand/v2/right/base_link.STL" />
+      </geometry>
+      <material
+        name="">
+        <color
+          rgba="0.792156862745098 0.819607843137255 0.933333333333333 1" />
+      </material>
+    </visual>
+    <collision>
+      <origin
+        xyz="0 0 0"
+        rpy="0 0 0" />
+      <geometry>
+        <mesh
+          filename="package://ur_description/meshes/inspire_hand/v2/right/base_link.STL" />
+      </geometry>
+    </collision>
+  </link>
+  <link
+    name="${prefix}right_thumb_swing">
+    <inertial>
+      <origin
+        xyz="-0.00178423179132727 0.000649410769092446 0.0048858931043441"
         rpy="0 0 0" />
       <mass
         value="0.00115518743162309" />
       <inertia
-        ixx="6.27834293959477E-08"
-        ixy="9.38445541803444E-10"
-        ixz="-3.50236810587605E-09"
-        iyy="3.78279141131513E-08"
-        iyz="-1.31528360070952E-10"
-        izz="6.1816168438865E-08" />
-    </inertial>
-    <visual>
-      <origin
-        xyz="0 0 0"
-        rpy="0 0 0" />
-      <geometry>
-        <mesh
-          filename="package://ur_description/meshes/inspire_hand/v2/left/left_thumb_swing.STL" />
-      </geometry>
-      <material
-        name="">
-        <color
-          rgba="0.792156862745098 0.819607843137255 0.933333333333333 1" />
-      </material>
-    </visual>
-    <collision>
-      <origin
-        xyz="0 0 0"
-        rpy="0 0 0" />
-      <geometry>
-        <mesh
-          filename="package://ur_description/meshes/inspire_hand/v2/left/left_thumb_swing.STL" />
+        ixx="5.98911473694572E-08"
+        ixy="-8.04324266712912E-09"
+        ixz="-3.29346964287941E-09"
+        iyy="4.07201940087006E-08"
+        iyz="1.1987242259973E-09"
+        izz="6.18161684388651E-08" />
+    </inertial>
+    <visual>
+      <origin
+        xyz="0 0 0"
+        rpy="0 0 0" />
+      <geometry>
+        <mesh
+          filename="package://ur_description/meshes/inspire_hand/v2/right/right_thumb_swing.STL" />
+      </geometry>
+      <material
+        name="">
+        <color
+          rgba="0.792156862745098 0.819607843137255 0.933333333333333 1" />
+      </material>
+    </visual>
+    <collision>
+      <origin
+        xyz="0 0 0"
+        rpy="0 0 0" />
+      <geometry>
+        <mesh
+          filename="package://ur_description/meshes/inspire_hand/v2/right/right_thumb_swing.STL" />
       </geometry>
     </collision>
@@ -93,55 +93,55 @@
     type="revolute">
     <origin
-      xyz="-0.035227 0.0908 -0.040206"
+      xyz="-0.035227 -0.0908 -0.041956"
       rpy="0 0 0" />
     <parent
       link="${prefix}hand_base_link" />
     <child
-      link="${prefix}left_thumb_swing" />
-    <axis
-      xyz="0 0 1" />
-    <limit
-      lower="0"
-      upper="1.70"
-      effort="1"
-      velocity="100" />
-  </joint>
-  <link
-    name="${prefix}left_thumb_1">
-    <inertial>
-      <origin
-        xyz="-0.0163208309809786 0.00996672794459635 -0.00940273641037634"
-        rpy="0 0 0" />
-      <mass
-        value="0.035" />
-      <inertia
-        ixx="1.05252775356938E-06"
-        ixy="8.8013589531825E-08"
-        ixz="4.12297543062756E-10"
-        iyy="1.12456993863274E-06"
-        iyz="-3.58528262599009E-10"
-        izz="1.43633392322177E-06" />
-    </inertial>
-    <visual>
-      <origin
-        xyz="0 0 0"
-        rpy="0 0 0" />
-      <geometry>
-        <mesh
-          filename="package://ur_description/meshes/inspire_hand/v2/left/left_thumb_1.STL" />
-      </geometry>
-      <material
-        name="">
-        <color
-          rgba="0.792156862745098 0.819607843137255 0.933333333333333 1" />
-      </material>
-    </visual>
-    <collision>
-      <origin
-        xyz="0 0 0"
-        rpy="0 0 0" />
-      <geometry>
-        <mesh
-          filename="package://ur_description/meshes/inspire_hand/v2/left/left_thumb_1.STL" />
+      link="${prefix}right_thumb_swing" />
+    <axis
+      xyz="0 0 -1" />
+    <limit
+      lower="0"
+      upper="1.7"
+      effort="1"
+      velocity="100" />
+  </joint>
+  <link
+    name="${prefix}right_thumb_1">
+    <inertial>
+      <origin
+        xyz="0.0161097484383394 0.0103028022975375 -0.00905330600289518"
+        rpy="0 0 0" />
+      <mass
+        value="0.030" />
+      <inertia
+        ixx="1.05608173707368E-06"
+        ixy="-8.93990422826739E-08"
+        ixz="-4.0717047155279E-10"
+        iyy="1.12055666436187E-06"
+        iyz="-3.12541187909307E-10"
+        izz="1.43604602983943E-06" />
+    </inertial>
+    <visual>
+      <origin
+        xyz="0 0 0"
+        rpy="0 0 0" />
+      <geometry>
+        <mesh
+          filename="package://ur_description/meshes/inspire_hand/v2/right/right_thumb_1.STL" />
+      </geometry>
+      <material
+        name="">
+        <color
+          rgba="0.792156862745098 0.819607843137255 0.933333333333333 1" />
+      </material>
+    </visual>
+    <collision>
+      <origin
+        xyz="0 0 0"
+        rpy="0 0 0" />
+      <geometry>
+        <mesh
+          filename="package://ur_description/meshes/inspire_hand/v2/right/right_thumb_1.STL" />
       </geometry>
     </collision>
@@ -151,70 +151,70 @@
     type="revolute">
     <origin
-      xyz="-0.0096402 -0.0097687 0.00125"
-      rpy="1.5708 0 0.037536" />
-    <parent
-      link="${prefix}left_thumb_swing" />
-    <child
-      link="${prefix}left_thumb_1" />
-    <axis
-      xyz="0 0 -1" />
-    <limit
-      lower="0"
-      upper="0.92"
-      effort="1"
-      velocity="100" />
-  </joint>
-  <link
-    name="${prefix}left_thumb_2">
-    <inertial>
-      <origin
-        xyz="-0.0100669921030146 0.0027226860312175 -0.00854141424002414"
-        rpy="0 0 0" />
-      <mass
-        value="0.023" />
-      <inertia
-        ixx="4.61650984659959E-07"
-        ixy="6.02617854200335E-08"
-        ixz="4.49999330286846E-11"
-        iyy="4.2100553287784E-07"
-        iyz="-2.1886405983307E-10"
-        izz="4.38695633575155E-07" />
-    </inertial>
-    <visual>
-      <origin
-        xyz="0 0 0"
-        rpy="0 0 0" />
-      <geometry>
-        <mesh
-          filename="package://ur_description/meshes/inspire_hand/v2/left/left_thumb_2.STL" />
-      </geometry>
-      <material
-        name="">
-        <color
-          rgba="0.792156862745098 0.819607843137255 0.933333333333333 1" />
-      </material>
-    </visual>
-    <collision>
-      <origin
-        xyz="0 0 0"
-        rpy="0 0 0" />
-      <geometry>
-        <mesh
-          filename="package://ur_description/meshes/inspire_hand/v2/left/left_thumb_2.STL" />
-      </geometry>
-    </collision>
-  </link>
-  <joint
-    name="${prefix}left_thumb_2_joint"
-    type="revolute">
-    <origin
-      xyz="-0.0385855343215257 0.0137354280979689 -0.00085000000007604"
+      xyz="-0.0063016 0.011924 0.003"
+      rpy="1.5708 0 2.7925" />
+    <parent
+      link="${prefix}right_thumb_swing" />
+    <child
+      link="${prefix}right_thumb_1" />
+    <axis
+      xyz="0 0 1" />
+    <limit
+      lower="0.035"
+      upper="0.90"
+      effort="1"
+      velocity="100" />
+  </joint>
+  <link
+    name="${prefix}right_thumb_2">
+    <inertial>
+      <origin
+        xyz="0.00924505131715823 0.00481918438391222 -0.00753905171750578"
+        rpy="0 0 0" />
+      <mass
+        value="0.020" />
+      <inertia
+        ixx="4.84948263631248E-07"
+        ixy="-4.6215685121335E-08"
+        ixz="-5.73077020148322E-11"
+        iyy="3.97628031594582E-07"
+        iyz="-2.99889919786187E-10"
+        izz="4.38765869483229E-07" />
+    </inertial>
+    <visual>
+      <origin
+        xyz="0 0 0"
+        rpy="0 0 0" />
+      <geometry>
+        <mesh
+          filename="package://ur_description/meshes/inspire_hand/v2/right/right_thumb_2.STL" />
+      </geometry>
+      <material
+        name="">
+        <color
+          rgba="0.792156862745098 0.819607843137255 0.933333333333333 1" />
+      </material>
+    </visual>
+    <collision>
+      <origin
+        xyz="0 0 0"
+        rpy="0 0 0" />
+      <geometry>
+        <mesh
+          filename="package://ur_description/meshes/inspire_hand/v2/right/right_thumb_2.STL" />
+      </geometry>
+    </collision>
+  </link>
+  <joint
+    name="${prefix}right_thumb_2_joint"
+    type="revolute">
+    <origin
+      xyz="0.038292 0.014535 -0.0015"
       rpy="0 0 0" />
     <parent
-      link="${prefix}left_thumb_1" />
-    <child
-      link="${prefix}left_thumb_2" />
-    <axis
-      xyz="0 0 -1" />
+      link="${prefix}right_thumb_1" />
+    <child
+      link="${prefix}right_thumb_2" />
+    <axis
+      xyz="0 0 1" />
     <limit
       lower="0"
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